Commit message: Add ARX5 MuJoCo sim-to-sim alignment

File: source/uwlab_assets/uwlab_assets/robots/arx5/assets/arx5.urdf (robot description, URDF)
Before this commit: robot X5A, 11 links, 10 joints
Joints:
- joint joint6: limit lower=-3.14 upper=3.14 effort=100 velocity=1000 -> lower=-1.5708 upper=1.5708 effort=100 velocity=1000

File: source/uwlab_assets/uwlab_assets/robots/arx5/assets/arx5_colored.urdf (robot description, URDF)
Before this commit: robot X5A, 11 links, 10 joints
Joints:
- joint joint6: limit lower=-3.14 upper=3.14 effort=100 velocity=1000 -> lower=-1.5708 upper=1.5708 effort=100 velocity=1000
